Commit message: Final URDF

File: mybot/urdf/mybot.xacro (robot description, xacro)
@@ -9,6 +9,5 @@
 	<xacro:property name="robot_wheel_mass" value="5"/>
 	<xacro:property name="robot_wheel_length" value="0.05"/>
-	<xacro:property name="robot_wheel_radius" value="0.1"/>
-	<xacro:property name="camera_mass" value="0.1"/>
+	<xacro:property name="robot_wheel_radius" value="0.15"/>
 	<xacro:property name="hokoyu_mass" value="1e-5"/>
 	<!-- Make Chassis of Bot -->
@@ -27,5 +26,5 @@
 			<origin xyz="0 0 0.05" rpy=" 0 0 0"/>
 			<geometry>
-				<box size="0.5 0.5 0.2"/>
+				<box size=".7 .5 .2"/>
 			</geometry>
 		</collision>
@@ -33,5 +32,5 @@
 			<origin xyz="0 0 0.05" rpy=" 0 0 0"/>
 			<geometry>
-				<box size="0.5 0.5 0.2"/>
+				<box size=".7 .5 .2"/>
 			</geometry>
 		</visual>
@@ -130,28 +129,4 @@
 			<geometry>
 				<cylinder radius="${robot_wheel_radius}" length="${robot_wheel_length}"/>
-			</geometry>
-		</collision>
-	</link>
-	<!-- Camera -->
-	<link name="camera">
-		<inertial>
-			<mass value="${camera_mass}"/>
-			<origin xyz="0 0 0" rpy="0 0 0"/>
-			<inertia
-		        ixx="1e-6" ixy="0.0" ixz="0.0"
-		        iyy="1e-6" iyz="0.0"
-		        izz="1e-6"
-		      />
-		</inertial>
-		<visual>
-			<origin xyz="0 0 0" rpy="0 0 0"/>
-			<geometry>
-				<box size="0.05 0.05 0.05"/>
-			</geometry>
-		</visual>
-		<collision>
-			<origin xyz="0 0 0" rpy="0 0 0"/>
-			<geometry>
-				<box size="0.05 0.05 0.05"/>
 			</geometry>
 		</collision>
@@ -220,11 +195,4 @@
 	    <dynamics damping="1.0" friction="1.0" />
 	</joint>
-	<!-- Camera Joint -->
-	<joint name="camera_joint" type="fixed">
-		<origin xyz="0.26 0 0" rpy="0 0 0" />
-		<parent link="chassis"/>
-		<child link="camera" />
-		<axis xyz="0 1 0"/>
-	</joint>
 	<!-- Hokoyu Joint -->
 	<joint name="hokuyo_joint" type="fixed">
@@ -241,5 +209,5 @@
 	<!-- Color of bot -->
 	<gazebo reference="left_wheel_front">
-		<material>Gazebo/Green</material>
+		<material>Gazebo/Orange</material>
 		<kp>1000000.0</kp> <!-- kp and kd for rubber -->
 		<kd>100.0</kd>
@@ -250,5 +218,5 @@
 	</gazebo>
 	<gazebo reference="left_wheel_back">
-		<material>Gazebo/Green</material>
+		<material>Gazebo/Orange</material>
 		<kp>1000000.0</kp> <!-- kp and kd for rubber -->
 		<kd>100.0</kd>
@@ -259,5 +227,5 @@
 	</gazebo>
 	<gazebo reference="right_wheel_front">
-		<material>Gazebo/Green</material>
+		<material>Gazebo/Orange</material>
 		<kp>1000000.0</kp> <!-- kp and kd for rubber -->
 		<kd>100.0</kd>
@@ -268,20 +236,14 @@
 	</gazebo>
 	<gazebo reference="right_wheel_back">
-		<material>Gazebo/Green</material>
-		<kp>1000000.0</kp> <!-- kp and kd for rubber -->
-		<kd>100.0</kd>
-		<mu1>1.0</mu1>
-		<mu2>1.0</mu2>
-		<maxVel>1.0</maxVel>
-		<minDepth>0.00</minDepth>
-	</gazebo>
-	<!--<gazebo reference="right_wheel">
-		<material>Gazebo/Green</material>
-	</gazebo>-->
-	<gazebo reference="camera">
+		<material>Gazebo/Orange</material>
+		<kp>1000000.0</kp> <!-- kp and kd for rubber -->
+		<kd>100.0</kd>
+		<mu1>1.0</mu1>
+		<mu2>1.0</mu2>
+		<maxVel>1.0</maxVel>
+		<minDepth>0.00</minDepth>
+	</gazebo>
+	<gazebo reference="chassis">
 		<material>Gazebo/Red</material>
-	</gazebo>
-	<gazebo reference="chassis">
-		<material>Gazebo/Blue</material>
 	</gazebo>
 	<!-- Motor, Camera and Lidar Simulation -->
